File: PassiveMultiples/PassiveMultiples.kicad_pcb (KiCad board)
At the start: 2 copper layers, 15 x 100 mm, 9 parts, among them J1 AudioJack2_SwitchT, J2 AudioJack2_SwitchT, J3 AudioJack2_SwitchT, J4 AudioJack2_SwitchT, J5 AudioJack2_SwitchT, J6 AudioJack2_SwitchT, J7 AudioJack2_SwitchT, J8 AudioJack2_SwitchT, SW1 SW_Push_DPDT

Commit message: Add ST-01 part number and CC BY-NC-SA mark to the main PCB
Four CC badges (Attribution, NonCommercial, ShareAlike, and the
Creative Commons roundel) as real footprint instances from
_NTSFootprints, not hand-drawn graphics, split across two rows so
they clear the neighboring jacks. ST-01 and the CC BY-NC-SA 4.0 text
moved to their own gap. The existing Passive Multiple/schenktronics.com
text was repositioned, not removed. Verified centered and square
against the board's true centerline with a calibrated render.
Parts:
- added G***: LOGO, _NTSFootprints:SchentronicsLogoSmed, B.Cu at (157.6, 49.8)
- added REF**: Symbol_CC-Attribution_SilkTop_Small, _NTSFootprints:Symbol_CC-Attribution_SilkTop_Small, B.Cu at (154.7, 105.0)
- added REF**: Symbol_CreativeCommons_SilkTop_Small, _NTSFootprints:Symbol_CreativeCommons_SilkTop_Small, B.Cu at (160.3, 105.0)
- added REF**: Symbol_CC-ShareAlike_SilkTop_Small, _NTSFootprints:Symbol_CC-ShareAlike_SilkTop_Small, B.Cu at (154.7, 117.0)
- added REF**: Symbol_CC-Noncommercial_SilkTop_Small, _NTSFootprints:Symbol_CC-Noncommercial_SilkTop_Small, B.Cu at (160.3, 117.0)
Other:
- net class Default removed
- board text added: "CC BY-NC-SA 4.0"
- board text added: "ST-01 v1.1 Passive Multiple"
- board text removed: "Passive Multiple v1.0"
