File: PassiveMultiples/PassiveMultiples.kicad_pcb (KiCad board)
At the start: 2 copper layers, 15 x 100 mm, 14 parts, among them J1 AudioJack2_SwitchT, J2 AudioJack2_SwitchT, J3 AudioJack2_SwitchT, J4 AudioJack2_SwitchT, J5 AudioJack2_SwitchT, J6 AudioJack2_SwitchT, J7 AudioJack2_SwitchT, J8 AudioJack2_SwitchT, SW1 SW_Push_DPDT

Commit message: Main PCB: drop the CC icon roundels, keep the license text
Nathan's own edit in KiCad: removed the four CC BY-NC-SA icon roundels
(Attribution/ShareAlike/Noncommercial/base), keeping just the
"CC BY-NC-SA 4.0" text line -- standardizing this board to match the
text-only convention the other three ended up on, where the icons
didn't reliably fit.
Parts:
- removed REF**: Symbol_CC-Attribution_SilkTop_Small, _NTSFootprints:Symbol_CC-Attribution_SilkTop_Small
- removed REF**: Symbol_CreativeCommons_SilkTop_Small, _NTSFootprints:Symbol_CreativeCommons_SilkTop_Small
- removed REF**: Symbol_CC-ShareAlike_SilkTop_Small, _NTSFootprints:Symbol_CC-ShareAlike_SilkTop_Small
- removed REF**: Symbol_CC-Noncommercial_SilkTop_Small, _NTSFootprints:Symbol_CC-Noncommercial_SilkTop_Small
