File: PassiveMultiplesFaceplate/PassiveMultiplesFaceplate.kicad_pcb (KiCad board)
At the start: 2 copper layers, 15 x 128.5 mm, 11 parts

Commit message: Update faceplate to new logo.  Regenerate gerbers.
Parts:
- added G***: LOGO, _NTSFootprints:SchentronicsLogo, F.Cu at (144.0, 170.5)
Routing:
- added copper zone on F.Cu, net (none)
Other:
- net class Default removed
- board text removed: "Schenk"

Commit message: Faceplate: S-mark + ST-01 moved to the hole-centered scheme, Orbitron text
S-mark moves from lower-left to the gap right of the bottom hole
(1.09mm margin each side) -- too narrow for the full wordmark, so this
is the small-mark branch of the new placement rule. ST-01 moves from
lower-right to the left gap, vertical, justify-left anchored to the
S-mark's bottom. Header and part number switched from italic KiCad
stroke font to upright Orbitron.

Note: this file carries other pending local changes from before this
edit, not just the faceplate update above.
Parts:
- removed the G*** at (144.0, 170.5)
- added G***: LOGO, _NTSFootprints:SchentronicsLogoSsmall, F.Cu at (155.2, 178.2)
Other:
- board text added: "ST-01"
